File: speedo-pcb/speedo-pcb.kicad_pcb (KiCad board)
At the start: 4 copper layers, 52 x 52 mm, 66 parts, among them J1 Debug, J2 Mode, J3 Speedo, J4 Power, J5 VBAT, J6 BOOT, J7 Breakout, M1 X27_128, U1 XC6206P332MR, U3 OLED_128x32, U4 STM32F103C8T6, U6 LGS5145, X2 Q13FC1350000400, X3 X322516MLB4SI

Commit message: Silence kibot W135 and mounting-hole warnings
Parts:
- renumbered REF** to H1, REF** to H2, REF** to H3, REF** to H4, REF** to H5, REF** to H6
Changed lines of the file:
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@@
 		(descr "Mounting Hole 2.2mm, M2")
 		(tags "mounting hole 2.2mm m2")
-		(property "Reference" "REF**"
+		(property "Reference" "H4"
 			(at 0 -3.2 0)
 			(layer "F.SilkS")
@@
 			)
 		)
-		(attr exclude_from_pos_files exclude_from_bom)
+		(attr board_only exclude_from_pos_files exclude_from_bom)
 		(fp_circle
 			(center 0 0)
@@
 		(descr "Mounting Hole 2.2mm, M2")
 		(tags "mounting hole 2.2mm m2")
-		(property "Reference" "REF**"
+		(property "Reference" "H1"
 			(at 0 -3.2 0)
 			(layer "F.SilkS")
@@
 			)
 		)
-		(attr exclude_from_pos_files exclude_from_bom)
+		(attr board_only exclude_from_pos_files exclude_from_bom)
 		(fp_circle
 			(center 0 0)
@@
 		(descr "Mounting Hole 2.2mm, M2")
 		(tags "mounting hole 2.2mm m2")
-		(property "Reference" "REF**"
+		(property "Reference" "H6"
 			(at 0 -3.2 0)
 			(layer "F.SilkS")
@@
 			)
 		)
-		(attr exclude_from_pos_files exclude_from_bom)
+		(attr board_only exclude_from_pos_files exclude_from_bom)
 		(fp_circle
 			(center 0 0)
@@
 		(descr "Mounting Hole 2.2mm, M2")
 		(tags "mounting hole 2.2mm m2")
-		(property "Reference" "REF**"
+		(property "Reference" "H2"
 			(at 0 -3.2 0)
 			(layer "F.SilkS")
@@
 			)
 		)
-		(attr exclude_from_pos_files exclude_from_bom)
+		(attr board_only exclude_from_pos_files exclude_from_bom)
 		(fp_circle
 			(center 0 0)
@@
 		(descr "Mounting Hole 2.2mm, M2")
 		(tags "mounting hole 2.2mm m2")
-		(property "Reference" "REF**"
+		(property "Reference" "H5"
 			(at 0 -3.2 0)
 			(layer "F.SilkS")
@@
 			)
 		)
-		(attr exclude_from_pos_files exclude_from_bom)
+		(attr board_only exclude_from_pos_files exclude_from_bom)
 		(fp_circle
 			(center 0 0)
@@
 		(descr "Mounting Hole 2.2mm, M2")
 		(tags "mounting hole 2.2mm m2")
-		(property "Reference" "REF**"
+		(property "Reference" "H3"
 			(at 0 -3.2 0)
 			(layer "F.SilkS")
@@
 			)
 		)
-		(attr exclude_from_pos_files exclude_from_bom)
+		(attr board_only exclude_from_pos_files exclude_from_bom)
 		(fp_circle
 			(center 0 0)
